File: Schematics/hvc/hvc-110_240_5174.kicad_sch (KiCad schematic)
At the start: 120 parts, among them J1 DIN41612_01x32_A, Q1 BC337, Q2 BC337, Q3 BC337, Q4 BC337, Q5 BC337, Q6 BC337, Q7 BC337, Q8 BC337, Q9 BC337

Commit message: Add files via upload
Connections:
- net at C4.2: now also IC4.8 (Comp_2)
- net at IC7.8 (Comp_2): now also C7.2
- net at C3.2: now also IC3.8 (Comp_2)
- net at C6.2: now also IC6.8 (Comp_2)
- net at C5.2: now also IC5.8 (Comp_2)
Changed lines of the file:
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@@
 	(wire
 		(pts
+			(xy 189.23 82.55) (xy 191.77 82.55)
+		)
+		(stroke
+			(width 0)
+			(type default)
+		)
+	)
+	(wire
+		(pts
 			(xy 262.89 16.51) (xy 262.89 21.59)
 		)
@@
 	(wire
 		(pts
+			(xy 133.35 81.28) (xy 133.35 82.55)
+		)
+		(stroke
+			(width 0)
+			(type default)
+		)
+	)
+	(wire
+		(pts
 			(xy 195.58 38.1) (xy 195.58 36.83)
 		)
@@
 	(wire
 		(pts
+			(xy 252.73 93.98) (xy 252.73 82.55)
+		)
+		(stroke
+			(width 0)
+			(type default)
+		)
+	)
+	(wire
+		(pts
 			(xy 173.99 165.1) (xy 173.99 196.85)
 		)
@@
 	(wire
 		(pts
+			(xy 133.35 82.55) (xy 132.08 82.55)
+		)
+		(stroke
+			(width 0)
+			(type default)
+		)
+	)
+	(wire
+		(pts
 			(xy 29.21 43.18) (xy 36.83 43.18)
 		)
@@
 	(wire
 		(pts
+			(xy 243.84 93.98) (xy 252.73 93.98)
+		)
+		(stroke
+			(width 0)
+			(type default)
+		)
+	)
+	(wire
+		(pts
 			(xy 209.55 156.21) (xy 210.82 156.21)
 		)
@@
 	(wire
 		(pts
+			(xy 162.56 93.98) (xy 162.56 82.55)
+		)
+		(stroke
+			(width 0)
+			(type default)
+		)
+	)
+	(wire
+		(pts
 			(xy 111.76 99.06) (xy 111.76 92.71)
 		)
@@
 	(wire
 		(pts
+			(xy 182.88 93.98) (xy 191.77 93.98)
+		)
+		(stroke
+			(width 0)
+			(type default)
+		)
+	)
+	(wire
+		(pts
 			(xy 92.71 109.22) (xy 54.61 109.22)
 		)
@@
 	(wire
 		(pts
+			(xy 252.73 82.55) (xy 250.19 82.55)
+		)
+		(stroke
+			(width 0)
+			(type default)
+		)
+	)
+	(wire
+		(pts
 			(xy 195.58 34.29) (xy 194.31 34.29)
 		)
@@
 	(wire
 		(pts
+			(xy 152.4 93.98) (xy 162.56 93.98)
+		)
+		(stroke
+			(width 0)
+			(type default)
+		)
+	)
+	(wire
+		(pts
 			(xy 120.65 26.67) (xy 124.46 26.67)
 		)
@@
 	(wire
 		(pts
+			(xy 162.56 82.55) (xy 160.02 82.55)
+		)
+		(stroke
+			(width 0)
+			(type default)
+		)
+	)
+	(wire
+		(pts
 			(xy 71.12 157.48) (xy 71.12 172.72)
 		)
@@
 	(wire
 		(pts
+			(xy 133.35 93.98) (xy 133.35 86.36)
+		)
+		(stroke
+			(width 0)
+			(type default)
+		)
+	)
+	(wire
+		(pts
 			(xy 217.17 113.03) (xy 217.17 105.41)
 		)
@@
 	(wire
 		(pts
+			(xy 220.98 83.82) (xy 220.98 82.55)
+		)
+		(stroke
+			(width 0)
+			(type default)
+		)
+	)
+	(wire
+		(pts
 			(xy 62.23 193.04) (xy 111.76 193.04)
 		)
@@
 	(wire
 		(pts
+			(xy 223.52 83.82) (xy 220.98 83.82)
+		)
+		(stroke
+			(width 0)
+			(type default)
+		)
+	)
+	(wire
+		(pts
 			(xy 66.04 167.64) (xy 66.04 165.1)
 		)
@@
 	(wire
 		(pts
+			(xy 213.36 93.98) (xy 222.25 93.98)
+		)
+		(stroke
+			(width 0)
+			(type default)
+		)
+	)
+	(wire
+		(pts
 			(xy 13.97 111.76) (xy 13.97 87.63)
 		)
@@
 	(wire
 		(pts
+			(xy 139.7 81.28) (xy 133.35 81.28)
+		)
+		(stroke
+			(width 0)
+			(type default)
+		)
+	)
+	(wire
+		(pts
 			(xy 104.14 66.04) (xy 104.14 60.96)
 		)
@@
 	(wire
 		(pts
+			(xy 222.25 86.36) (xy 223.52 86.36)
+		)
+		(stroke
+			(width 0)
+			(type default)
+		)
+	)
+	(wire
+		(pts
 			(xy 96.52 154.94) (xy 96.52 140.97)
 		)
@@
 	(wire
 		(pts
+			(xy 222.25 93.98) (xy 222.25 86.36)
+		)
+		(stroke
+			(width 0)
+			(type default)
+		)
+	)
+	(wire
+		(pts
 			(xy 238.76 93.98) (xy 226.06 93.98)
 		)
@@
 	(wire
 		(pts
+			(xy 124.46 93.98) (xy 133.35 93.98)
+		)
+		(stroke
+			(width 0)
+			(type default)
+		)
+	)
+	(wire
+		(pts
 			(xy 219.71 113.03) (xy 219.71 115.57)
 		)
@@
 	(wire
 		(pts
+			(xy 139.7 86.36) (xy 139.7 81.28)
+		)
+		(stroke
+			(width 0)
+			(type default)
+		)
+	)
+	(wire
+		(pts
 			(xy 29.21 83.82) (xy 48.26 83.82)
 		)
@@
 	(wire
 		(pts
+			(xy 220.98 82.55) (xy 219.71 82.55)
+		)
+		(stroke
+			(width 0)
+			(type default)
+		)
+	)
+	(wire
+		(pts
 			(xy 29.21 147.32) (xy 48.26 147.32)
 		)
@@
 	(wire
 		(pts
+			(xy 191.77 93.98) (xy 191.77 82.55)
+		)
+		(stroke
+			(width 0)
+			(type default)
+		)
+	)
+	(wire
+		(pts
 			(xy 182.88 29.21) (xy 182.88 44.45)
 		)
@@
 		)
 		(stroke
+			(width 0)
+			(type default)
+		)
+	)
+	(wire
+		(pts
+			(xy 133.35 86.36) (xy 139.7 86.36)
+		)
+		(stroke
+			(width 0)
+			(type default)
+		)
+	)
+	(wire
+		(pts
+			(xy 223.52 86.36) (xy 223.52 83.82)
+		)
+		(stroke

Commit message: Add files via upload
Connections:
- net at D9.1 (K), IC7.2 (Input-), JP1.2 (B)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: now also R43.2
- net at Q2.2 (B), R2.1: now also D2.1 (K), R4.1
- net at IC6.2 (Input-), R39.1, R46.2: now also R45.2
- net at D11.1 (K): now also R60.1
- net at C8.2, D11.2 (A): now also R54.2
- net at R48.2: now also K3.1 (In)
- net at J1.a14 (Pin_a14): now also R57.2
- net at Q3.2 (B), R8.2: now also D4.1 (K), R10.2
- net at Q6.2 (B), R19.2: now also D8.1 (K), R21.2
- net at Q5.2 (B), R13.1: now also D6.1 (K), R15.1
- net at K2.1 (In): now also R37.2
- net at K5.1 (In), R61.1: now also R50.2
- net at R35.2: now also K4.8 (Out), R34.2
- net at K6.8 (Out): now also R51.2, R52.2
